Commit message: fix wheelwalker urdf

File: resources/robots/wheelwalker/urdf/wheelwalker_v1.urdf (robot description, URDF)
Before this commit: robot wheelwalker_v1, 17 links, 16 joints
Links:
- link base_link: geometry collision box size=0.27 0.24 0.35; visual mesh filename=../meshes/wheelwalker_v0.1/base_link.stl
- link left_foot_link: geometry collision cylinder length=0.18 radius=0.012; visual mesh filename=../meshes/wheelwalker_v0.1/left_foot_link.stl scale=0.001 0.001 0.001
- link left_hip_pitch_link: geometry collision cylinder length=0.08879999999999999 radius=0.0185; visual mesh filename=../meshes/wheelwalker_v0.1/left_hip_pitch_link.stl scale=0.001 0.001 0.001
- link left_hip_roll_link: geometry collision cylinder length=0.08879999999999999 radius=0.0185; visual mesh filename=../meshes/wheelwalker_v0.1/left_hip_roll_link.stl scale=0.001 0.001 0.001
- link left_hip_yaw_link: geometry collision cylinder length=0.08879999999999999 radius=0.0185; visual mesh filename=../meshes/wheelwalker_v0.1/left_hip_yaw_link.stl scale=0.001 0.001 0.001
- link left_thigh_link: geometry collision cylinder length=0.25 radius=0.033; visual mesh filename=../meshes/wheelwalker_v0.1/left_thigh_link.stl scale=0.001 0.001 0.001
- link left_tibia_link: geometry collision cylinder length=0.25 radius=0.0315; visual mesh filename=../meshes/wheelwalker_v0.1/left_tibia_link.stl scale=0.001 0.001 0.001
- link left_wheel_link: geometry collision cylinder length=0.03 radius=0.11; visual mesh filename=../meshes/wheelwalker_v0.1/left_wheel_link.stl scale=0.001 0.001 0.001
- link right_foot_link: geometry collision cylinder length=0.18 radius=0.012; visual mesh filename=../meshes/wheelwalker_v0.1/right_foot_link.stl scale=0.001 0.001 0.001
- link right_hip_pitch_link: geometry collision cylinder length=0.08879999999999999 radius=0.0185; visual mesh filename=../meshes/wheelwalker_v0.1/right_hip_pitch_link.stl scale=0.001 0.001 0.001
- link right_hip_roll_link: geometry collision cylinder length=0.08879999999999999 radius=0.0185; visual mesh filename=../meshes/wheelwalker_v0.1/right_hip_roll_link.stl scale=0.001 0.001 0.001
- link right_hip_yaw_link: geometry collision cylinder length=0.08879999999999999 radius=0.0185; visual mesh filename=../meshes/wheelwalker_v0.1/right_hip_yaw_link.stl scale=0.001 0.001 0.001
- link right_thigh_link: geometry collision cylinder length=0.25 radius=0.033; visual mesh filename=../meshes/wheelwalker_v0.1/right_thigh_link.stl scale=0.001 0.001 0.001
- link right_tibia_link: geometry collision cylinder length=0.25 radius=0.0315; visual mesh filename=../meshes/wheelwalker_v0.1/right_tibia_link.stl scale=0.001 0.001 0.001
- link right_wheel_link: geometry collision cylinder length=0.03 radius=0.11; visual mesh filename=../meshes/wheelwalker_v0.1/right_wheel_link.stl scale=0.001 0.001 0.001
- link tail_link: geometry collision box size=0.19 0.21 0.185; visual mesh filename=../meshes/wheelwalker_v0.1/tail_link.stl scale=0.001 0.001 0.001
Joints:
- joint tail_pitch_joint: type revolute -> fixed
